File: MacroV2/MacroPCBs/ads/ads.kicad_sch (KiCad schematic)
At the start: 46 parts, among them J1 Conn_01x15_Pin, SW1 RotaryEncoder_Switch, SW2 RotaryEncoder_Switch, SW3 SW_Push, U1 Raspberry_Pi_Pico

Commit message: PCB revisions, Newest is in production
Other:
- title: Macro PCB -> (none)
