File: MacroV2/MacroPCBs/macrov2.0.004/macrov2.0.004.kicad_sch (KiCad schematic)
At the start: 46 parts, among them J1 Conn_01x15_Pin, SW1 RotaryEncoder_Switch, SW2 RotaryEncoder_Switch, SW3 SW_Push, U1 Raspberry_Pi_Pico

Commit message: Added Zoom in and Zoom out funcs to encoder2
Parts:
- added D14: LED_SK6812MINI-E, ScottoKeebs_Components:LED_SK6812MINI-E, symbol ScottoKeebs:LED_SK6812MINI-E
Changed lines of the file:
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@@
+    )
+  )
+  (symbol (lib_id "ScottoKeebs:LED_SK6812MINI-E") (at 41.91 171.45 0) (unit 1)
+    (in_bom yes) (on_board yes) (dnp no) (fields_autoplaced)
+    (property "Reference" "D14" (at 41.91 161.29 0)
+      (effects (font (size 1.27 1.27)))
+    )
+    (property "Value" "LED_SK6812MINI-E" (at 41.91 163.83 0)
+      (effects (font (size 1.27 1.27)))
+    )
+    (property "Footprint" "ScottoKeebs_Components:LED_SK6812MINI-E" (at 43.18 179.07 0)
+      (effects (font (size 1.27 1.27)) (justify left top) hide)
+    )
+    (property "Datasheet" "https://cdn-shop.adafruit.com/product-files/2686/SK6812MINI_REV.01-1-2.pdf" (at 43.18 181.61 0)
+      (effects (font (size 1.27 1.27)) (justify left top) hide)
+    )
+    (pin "3")
+    (pin "4")
+    (pin "1")
+    (pin "2")
+    (instances
+      (project "macrov2.0.004"
+        (path "/4de1fd36-c486-4527-b451-b6db308c052e"
+          (reference "D14") (unit 1)
+        )
+      )
     )
   )
